Commit message: Fix logic to decide bot placement
- Fixed logic for determining placement of mobile base. Earlier bot was moving to slightly wrong position due to which ball was missed.
- Added property to make the racquet less stiff. Earlier ball was falling nearby after being hit by the racquet. Now it move away.

File: ros2/src/test_bot/description/arm2_core.xacro (robot description, xacro)
@@ -9,7 +9,7 @@
         <xacro:property name="l3_length" value="0.3"/>
         <xacro:property name="l4_length" value="0.15"/>
-        <xacro:property name="racquet_thickness" value="0.02"/>
-        <xacro:property name="racquet_radius" value="0.2"/>
-        <xacro:property name="general_mass" value="0.1"/>
+        <xacro:property name="racquet_thickness" value="0.07"/>     <!-- 0.02-->
+        <xacro:property name="racquet_radius" value="0.25"/>        <!-- 0.2-->
+        <xacro:property name="general_mass" value="0.1"/>           <!-- 0.1-->
         <xacro:property name="general_radius" value="0.02"/>
         <!-- MATERIALS -->
@@ -177,4 +177,14 @@
             <origin xyz="0 0 0" rpy="0 0 0"/>
         </xacro:link_macro>
+        <gazebo reference="racquet_link">
+            <mu1>0</mu1>
+            <mu2>0</mu2>
+            <!-- <kp>500000</kp> -->
+            <kp>50000</kp>
+            <kd>0</kd>
+            <minDepth>0</minDepth>
+            <maxVel>1000</maxVel>
+            <material>Gazebo/Blue</material>
+        </gazebo>
     </xacro:macro>
 </robot>

Commit message: Fix bot movement to goal
- The bot now moves to predicted point for hitting ball on time. Earlier the bot tends to overshoot the target.
- '__pycache__' folder which was accidently added has been removed.

File: ros2/src/test_bot/description/arm2_core.xacro (robot description, xacro)
@@ -5,5 +5,5 @@
         <!-- Variables -->
         <xacro:property name="sphere_radius" value="0.1"/>
-        <xacro:property name="sphere_mass" value="0.5"/>
+        <xacro:property name="sphere_mass" value="0.01"/>            <!-- 0.5-->
         <xacro:property name="l2_length" value="0.5"/>
         <xacro:property name="l3_length" value="0.3"/>
@@ -11,5 +11,5 @@
         <xacro:property name="racquet_thickness" value="0.07"/>     <!-- 0.02-->
         <xacro:property name="racquet_radius" value="0.25"/>        <!-- 0.2-->
-        <xacro:property name="general_mass" value="0.1"/>           <!-- 0.1-->
+        <xacro:property name="general_mass" value="0.01"/>           <!-- 0.1-->
         <xacro:property name="general_radius" value="0.02"/>
         <!-- MATERIALS -->

File: ros2/src/test_bot/description/mec_robot_core.xacro (robot description, xacro)
@@ -14,9 +14,9 @@
     <xacro:property name="chassis_height" value="0.6"/>      <!-- 6 meter = 600 cm -->
     <xacro:property name="chassis_depth" value="0.02"/>      <!-- 0.02meter = 2 cm -->
-    <xacro:property name="chassis_mass" value="1"/>          <!-- 1 kg -->
+    <xacro:property name="chassis_mass" value="0.1"/>          <!-- 1 kg -->
     <!-- Wheel Properties -->
     <xacro:property name="wheel_radius" value="0.02"/>
     <xacro:property name="wheel_width" value="0.02"/>
-    <xacro:property name="wheel_mass" value="1"/>
+    <xacro:property name="wheel_mass" value="0.1"/>               <!-- 1 kg -->
     <!-- Wheel Macro -->
     <xacro:macro name="wheel_macro" params="wheel_name wheel_color">    <!-- mu max_val=1 (max friction) min_val=0(min friction) -->
